File: usb_power/v1/usb_power.kicad_pcb (KiCad board)
At the start: 2 copper layers, 70.2 x 24.1 mm, 10 parts, among them J1 USB3_A, J2 Screw_Terminal_01x02, U1 MT3608

Commit message: what a pain
Parts:
- added U2: TPS55340PWPR, sulicat:IC_TPS55340PWPR, F.Cu at (161.8, 75.5)
- J1: footprint Connector_USB:USB3_A_Molex_48393-001 -> sulicat:USB3_MOLEX_0484050003
- ON/OFF1: footprint Button_Switch_THT:SW_DIP_SPSTx01_Slide_9.78x4.72mm_W7.62mm_P2.54mm -> sulicat:SW_DS01_254-L-01BE_CUD
- moved J2 66.4 mm to (122.9, 95.2), turned to 0 degrees
- moved R2 66.1 mm to (139.5, 86.8), turned to 0 degrees
- moved R1 61.3 mm to (139.5, 84.2)
- moved L1 59.3 mm to (140.4, 99.5), turned to 0 degrees
- moved U1 57.8 mm to (144.1, 85.2)
- moved RV1 56.6 mm to (142.8, 96.0)
- moved C1 55.1 mm to (134.8, 91.3), turned to 0 degrees
- moved C2 45.9 mm to (134.8, 96.2)
- moved ON/OFF1 39.1 mm to (139.5, 80.2), turned to 0 degrees
- moved J1 23.1 mm to (128.8, 76.3), turned to 0 degrees
Routing:
- net GND: track 96.4 -> 0.00 mm, vias 2 -> 0
- net Net-(J2-Pin_1): track 45.9 -> 0.00 mm
- net Net-(J1-VBUS): track 44.9 -> 0.00 mm
- net Net-(U1-FB): track 30.2 -> 0.00 mm, vias 2 -> 0
- net Net-(R2-Pad1): track 22.7 -> 0.00 mm, vias 2 -> 0
- net Net-(R1-Pad2): track 15.4 -> 0.00 mm, vias 2 -> 0
- net Net-(U1-EN): track 8.17 -> 0.00 mm
- net Net-(J1-D+): track 2.00 -> 0.00 mm
Other:
- board outline removed
