File: usb_power/v1/usb_power.kicad_sch (KiCad schematic)
At the start: 10 parts, among them J1 USB3_A, J2 Screw_Terminal_01x02, U1 MT3608

Commit message: fail, this is hard!
Parts:
- J1: Part Number (none) -> Molex 48393-0001
- U1: Part Number (none) -> MT3608 SOT23-6
Changed lines of the file:
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@@
+			)
+		)
+		(property "Part Number" "MT3608 SOT23-6"
+			(at 82.55 44.45 0)
+			(effects
+				(font
+					(size 1.27 1.27)
+				)
+				(hide yes)
 			)
 		)
@@
 			)
 		)
-		(property "Datasheet" "~"
+		(property "Datasheet" "https://www.molex.com/en-us/products/part-detail/483930001"
 			(at 46.99 49.53 0)
 			(effects
@@
 			)
 		)
+		(property "Part Number" "Molex   48393-0001 "
+			(at 43.18 52.07 0)
+			(effects
+				(font
+					(size 1.27 1.27)
+				)
+				(hide yes)
+			)
+		)

Commit message: what a pain
Parts:
- added U2: TPS55340PWPR, sulicat:IC_TPS55340PWPR, symbol sulicat:TPS55340PWPR
- J1: footprint Connector_USB:USB3_A_Molex_48393-001 -> sulicat:USB3_MOLEX_0484050003; Part Number Molex 48393-0001 -> Digikey WM25179-ND
- L1: footprint Inductor_SMD:L_0805_2012Metric -> sulicat:L_THT
- ON/OFF1: footprint Button_Switch_THT:SW_DIP_SPSTx01_Slide_9.78x4.72mm_W7.62mm_P2.54mm -> sulicat:SW_DS01_254-L-01BE_CUD
Changed lines of the file:
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@@
 			)
 		)
-		(property "Footprint" "Button_Switch_THT:SW_DIP_SPSTx01_Slide_9.78x4.72mm_W7.62mm_P2.54mm"
+		(property "Footprint" "sulicat:SW_DS01_254-L-01BE_CUD"
 			(at 68.58 62.23 0)
 			(effects
@@
 			)
 		)
-		(property "Footprint" "Inductor_SMD:L_0805_2012Metric"
+		(property "Footprint" "sulicat:L_THT"
 			(at 83.82 30.48 0)
 			(effects
@@
 			)
 		)
-		(property "Datasheet" "~"
+		(property "Datasheet" "https://www.digikey.com/en/products/detail/epcos-tdk-electronics/B78108S1105J000/652579"
 			(at 83.82 30.48 0)
 			(effects
@@
 	)
 	(symbol
+		(lib_id "sulicat:TPS55340PWPR")
+		(at 69.85 110.49 0)
+		(unit 1)
+		(exclude_from_sim no)
+		(in_bom yes)
+		(on_board yes)
+		(dnp no)
+		(fields_autoplaced yes)
+		(property "Reference" "U2"
+			(at 69.85 87.63 0)
+			(effects
+				(font
+					(size 1.27 1.27)
+				)
+			)
+		)
+		(property "Value" "TPS55340PWPR"
+			(at 69.85 90.17 0)
+			(effects
+				(font
+					(size 1.27 1.27)
+				)
+			)
+		)
+		(property "Footprint" "sulicat:IC_TPS55340PWPR"
+			(at 69.596 85.598 0)
+			(effects
+				(font
+					(size 1.27 1.27)
+				)
+				(justify bottom)
+				(hide yes)
+			)
+		)
+		(property "Datasheet" ""
+			(at 69.85 110.49 0)
+			(effects
+				(font
+					(size 1.27 1.27)
+				)
+				(hide yes)
+			)
+		)
+		(property "Description" ""
+			(at 69.85 110.49 0)
+			(effects
+				(font
+					(size 1.27 1.27)
+				)
+				(hide yes)
+			)
+		)
+		(property "PARTREV" "E"
+			(at 76.454 91.186 0)
+			(effects
+				(font
+					(size 1.27 1.27)
+				)
+				(justify bottom)
+				(hide yes)
+			)
+		)
+		(property "MANUFACTURER" "Texas Instruments"
+			(at 69.342 82.042 0)
+			(effects
+				(font
+					(size 1.27 1.27)
+				)
+				(justify bottom)
+				(hide yes)
+			)
+		)
+		(property "MAXIMUM_PACKAGE_HEIGHT" "1.2 mm"
+			(at 69.85 91.44 0)
+			(effects
+				(font
+					(size 1.27 1.27)
+				)
+				(justify bottom)
+				(hide yes)
+			)
+		)
+		(property "STANDARD" "Manufacturer recommendations"
+			(at 68.834 88.646 0)
+			(effects
+				(font
+					(size 1.27 1.27)
+				)
+				(justify bottom)
+				(hide yes)
+			)
+		)
+		(pin "7"
+		)
+		(pin "5"
+		)
+		(pin "14"
+		)
+		(pin "3"
+		)
+		(pin "18"
+		)
+		(pin "1"
+		)
+		(pin "10"
+		)
+		(pin "2"
+		)
+		(pin "6"
+		)
+		(pin "4"
+		)
+		(pin "13"
+		)
+		(pin "12"
+		)
+		(pin "8"
+		)
+		(pin "9"
+		)
+		(pin "20"
+		)
+		(pin "17"
+		)
+		(pin "11"
+		)
+		(pin "19"
+		)
+		(pin "15"
+		)
+		(pin "21"
+		)
+		(pin "16"
+		)
+		(instances
+			(project ""
+				(path "/a1545928-1195-40b9-b3c4-78f837012afb"
+					(reference "U2")
+					(unit 1)
+				)
+			)
+		)
+	)
+	(symbol
 		(lib_id "power:GND")
 		(at 105.41 88.9 0)
@@
 		(on_board yes)
 		(dnp no)
-		(fields_autoplaced yes)
 		(property "Reference" "J1"
 			(at 43.18 33.02 0)
@@
 			)
 		)
-		(property "Footprint" "Connector_USB:USB3_A_Molex_48393-001"
+		(property "Footprint" "sulicat:USB3_MOLEX_0484050003"
 			(at 46.99 49.53 0)
 			(effects
@@
 			)
 		)
-		(property "Datasheet" "https://www.molex.com/en-us/products/part-detail/483930001"
+		(property "Datasheet" "https://www.digikey.com/en/products/detail/molex/0484050004/6823026"
 			(at 46.99 49.53 0)
 			(effects
@@
 			)
 		)
-		(property "Description" ""
+		(property "Description" "CONN RCPT USB3.0 TYPEA 9POS R/A"
+			(at 42.164 28.956 0)
+			(effects
+				(font
+					(size 1.27 1.27)
+				)
+				(hide yes)
+			)
+		)
+		(property "Part Number" "Digikey WM25179-ND"
 			(at 43.18 52.07 0)
 			(effects
-				(font
-					(size 1.27 1.27)
-				)
-			)
-		)
-		(property "Part Number" "Molex   48393-0001 "
-			(at 43.18 52.07 0)
-			(effects
